Commit message: feat(stereo_mount): record ZED-M IMU at ~800Hz (SDK-free HID)
Add ZedImu: opens the ZED-M HID interface and replays the official SDK's
stream-start handshake (two output reports, captured via usbmon) instead of
zed-open-capture's feature-report + 250ms ping. That handshake is what avoids
the firmware's sporadic ~1s IMU stream suspensions — verified gap-free over a
16-min soak (774k samples @795Hz, max gap 3.75ms) with no SDK/CUDA.

Wire it into StereoMountRecorder (new zed_imu In stream, autoconnected) and add
a placeholder zed_imu_link frame to the rig URDF so recorded IMU resolves in tf.
Values validated live: 795Hz, |accel|~10.4 m/s^2 (raw factory-uncalibrated),
|gyro|~0.03 rad/s stationary.

File: dimos/robot/assembly/stereo_mount/stereo_mount.urdf (robot description, URDF)
Before this commit: robot stereo_mount, 9 links, 8 joints
Links:
- added link zed_imu_link
Joints:
- added joint zed_to_imu: type fixed, parent zed_link, child zed_imu_link, origin xyz=0 0.0315 0 rpy=0 0 0
