Commit message: r1lite: adopt the merged Pink teleop architecture (PR #3237)
Ports the teleop core as merged to main — cartesian_ik_task,
teleop_task, and eef_twist_task with their suites — onto the validated
r1lite deployment branch. The solver now owns smoothness (damping task,
velocity clamp) and safety (configuration limits with seed tolerance),
replacing the chase-window and step-gate machinery the old architecture
needed. The r1lite blueprint moves to the A1Z-parity configuration with
two field-informed deviations: timeout 1.5s rides through vendor
pose-stream gaps, and seed_limit_tolerance 0.05 rad covers the folded
boot pose measured up to 1.74 deg below the vendor URDF lower bound —
the merged default would still hard-fail there. The grasp-center TCP
(0.17 m past joint 6) becomes a fixed URDF frame on both arms, replacing
the removed task-level tool offset. The quest module keeps our session
recorder, which main does not carry. R1lite tests move to the new API:
engagement is required before pose deltas act, per-tick deltas bound by
the velocity clamp, and limit checks read the solver's runtime model.

File: dimos/robot/galaxea/r1lite/assets/r1lite_left_arm.urdf (robot description, URDF)
Before this commit: robot r1lite_left_arm, 7 links, 6 joints
Links:
- added link left_arm_grasp_center
Joints:
- added joint left_arm_grasp_center_joint: type fixed, parent left_arm_link6, child left_arm_grasp_center, origin xyz=0.17 0 0 rpy=0 0 0

File: dimos/robot/galaxea/r1lite/assets/r1lite_right_arm.urdf (robot description, URDF)
Before this commit: robot r1lite_right_arm, 7 links, 6 joints
Links:
- added link right_arm_grasp_center
Joints:
- added joint right_arm_grasp_center_joint: type fixed, parent right_arm_link6, child right_arm_grasp_center, origin xyz=0.17 0 0 rpy=0 0 0
